File: micro/stlinkv2.kicad_pcb (KiCad board)
At the start: 2 copper layers, 60 parts, among them J1 TX, J2 RX, J3 JTAG, J4 SWIMM, J5 USB_B, U1 AZ1117-3.3, U2 STM32F103C8Tx, Y1 8M

Commit message: micro usb
Parts:
- D2: moved to B.Cu
- J3: footprint stlinkv2:PinSocket_2x10_P2.54mm_Vertical -> micro:PinSocket_2x10_P2.54mm_Vertical
- J5: value USB_B -> USB_B_Micro; footprint Connector_USB:USB_B_OST_USB-B1HSxx_Horizontal -> Connector_USB:USB_Micro-B_Amphenol_10104110_Horizontal
- moved D12 17.0 mm to (112.1, 46.1), turned to 270 degrees
- moved D10 10.3 mm to (114.2, 57.0), turned to 90 degrees
- moved J2 6.94 mm to (111.1, 42.4)
- moved D2 6.15 mm to (110.2, 52.7), turned to 90 degrees
- moved J5 3.24 mm to (109.7, 52.0), turned to 270 degrees
- moved R1 1.10 mm to (113.0, 52.8)
- moved J1 0.91 mm to (111.1, 38.3)
Connections:
- D2 pad : GND -> (no net)
- J5 pad 4: GND -> Net-(J5-Pad4)
Routing:
- net (no net): track 480.0 -> 0.00 mm
- net GND: track 488.8 -> 462.3 mm
- net Net-(D12-Pad1): track 26.6 -> 10.3 mm
- net Net-(D10-Pad1): track 23.2 -> 8.70 mm
- net Net-(J2-Pad1): track 23.9 -> 15.5 mm
- net Net-(D2-Pad1): track 13.3 -> 9.52 mm, vias 0 -> 1
- net +3V3: track 62.3 -> 60.1 mm
