File: wire/stlinkv2.kicad_pcb (KiCad board)
At the start: 2 copper layers, 61 parts, among them J1 TX, J2 RX, J3 JTAG, J4 SWIMM, J5 USB_B, U1 AZ1117-3.3, U2 STM32F103C8Tx, Y1 8M

Commit message: tested
Parts:
- removed R25: 75, Resistor_SMD:R_0805_2012Metric_Pad1.15x1.40mm_HandSolder
- D2: moved to B.Cu
- J3: footprint stlinkv2:PinSocket_2x10_P2.54mm_Vertical -> micro:PinSocket_2x10_P2.54mm_Vertical
- J5: value USB_B -> Conn_01x04; footprint Connector_USB:USB_B_OST_USB-B1HSxx_Horizontal -> Connector_Wire:SolderWire-0.25sqmm_1x04_P4.5mm_D0.65mm_OD2mm
- moved D12 17.6 mm to (113.5, 46.7)
- moved D10 10.3 mm to (114.2, 57.0), turned to 90 degrees
- moved J5 10.0 mm to (110.1, 59.7), turned to 90 degrees
- moved R1 7.70 mm to (117.1, 59.5), turned to 0 degrees
- moved J2 6.94 mm to (111.1, 42.4)
- moved D2 2.70 mm to (113.5, 60.3), turned to 90 degrees
- moved J1 0.91 mm to (111.1, 38.3)
Connections:
- D3 pad : GND -> (no net)
- D8 pad : GND -> (no net)
- J5 pad 2: Net-(D12-Pad1) -> Net-(D10-Pad1)
- J5 pad 3: Net-(D10-Pad1) -> Net-(D12-Pad1)
Routing:
- net (no net): track 480.0 -> 0.00 mm
- net Net-(J2-Pad1): track 54.3 -> 16.0 mm, vias 1 -> 0
- net GND: track 479.9 -> 451.1 mm
- net Net-(D12-Pad1): track 26.6 -> 8.51 mm
- net Net-(D10-Pad1): track 23.2 -> 9.57 mm
- net VBUS: track 39.4 -> 28.7 mm
- net +3V3: track 69.5 -> 60.1 mm
- net Net-(D2-Pad1): track 13.3 -> 6.28 mm
- net /TDO_SWO: track 43.0 -> 40.2 mm, vias 1 -> 0
- net /LED: track 23.4 -> 24.7 mm
Other:
- board text removed: "RX"
- board text removed: "TX"
